File: Signals/Signals.kicad_sch (KiCad schematic)
At the start: 32 parts, among them J1 IN, J2 IN, J3 OUT, J4 OUT, J5 IN, J6 IN, J7 OUT, J8 OUT, J9 Power, U1 TL074

Commit message: Update Signals.kicad_sch
Connections:
- net +12V: now also C1.2
Other:
- note added: "power protection needed"
Changed lines of the file:
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@@
   (junction (at 123.19 96.52) (diameter 0) (color 0 0 0 0)
+  )
+  (junction (at 50.8 135.89) (diameter 0) (color 0 0 0 0)
   )
   (junction (at 72.39 135.89) (diameter 0) (color 0 0 0 0)
@@
     (stroke (width 0) (type default) (color 0 0 0 0))
   )
+  (wire (pts (xy 50.8 133.35) (xy 50.8 135.89))
+    (stroke (width 0) (type default) (color 0 0 0 0))
+  )
   (wire (pts (xy 234.95 99.06) (xy 236.22 99.06))
     (stroke (width 0) (type default) (color 0 0 0 0))
@@
     (stroke (width 0) (type default) (color 0 0 0 0))
   )
+  (text "power protection needed" (at 59.69 128.27 0)
+    (effects (font (size 1.27 1.27) (thickness 0.254) bold) (justify left bottom))
+  )
   (symbol (lib_id "Device:R") (at 236.22 48.26 90) (unit 1)

Commit message: Power updates!
Parts:
- added D5, D6: 1N5817, Diode_THT:D_DO-41_SOD81_P10.16mm_Horizontal, symbol Diode:1N5817
- 10k1, 10k2, 10k3, 10k4: footprint (none) -> Potentiometer_THT:Potentiometer_Alpha_RD901F-40-00D_Single_Vertical
- C1, C2: footprint (none) -> Capacitor_THT:C_Disc_D5.0mm_W2.5mm_P5.00mm
- D1, D2, D3, D4: footprint (none) -> LED_THT:LED_D3.0mm
- J9: footprint (none) -> Connector_PinSocket_2.54mm:PinSocket_2x05_P2.54mm_Vertical
- R1, R10, R11, R12, R2, R3, R4, R5, R6, R7, R8, R9: footprint (none) -> Resistor_THT:R_Axial_DIN0207_L6.3mm_D2.5mm_P10.16mm_Horizontal
- U1: footprint (none) -> Package_DIP:DIP-14_W7.62mm_LongPads
Connections:
- net +12V: now also D6.2 (A); no longer C1.2, U1.4 (V+)
- net -12V: now also D5.1 (K); no longer C2.1, U1.11 (V-)
- new net: C2.1, D5.2 (A), U1.11 (V-)
- new net: C1.2, D6.1 (K), U1.4 (V+)
Other:
- note added: "schottky diodes for reverse current protection"
- note removed: "power protection needed"
- company: (none) -> formation electronics
- title: (none) -> Signals
